File: rev1.a/retroii/video.sch (KiCad schematic (older format))
At the start: 29 parts, among them J1 VGA, P1 PROP_PLUG, SW1 SW_PUSH_SAFE, U4 Prop_P8X32A, U5 24LC256_EEPROM, Y1 5MHz 20pf

Commit message: added vga dsub-15 footprint and 3d model
Parts:
- J1: footprint 6502Library:117343442VGA -> retroii_footprints:Amphenol_ICD15S13E6GV00LF
Changed lines of the file:
@@
 F 0 "J1" H 6960 6300 60  0000 C CNN
 F 1 "VGA" H 7210 4750 60  0000 C CNN
-F 2 "6502Library:117343442VGA" H 7210 5500 60  0001 C CNN
+F 2 "retroii_footprints:Amphenol_ICD15S13E6GV00LF" H 7210 5500 60  0001 C CNN
 F 3 "" H 7210 5500 60  0000 C CNN
 	1    7210 5500

Commit message: added tactile switches 3d models, footprints, symbols.
Parts:
- SW1: footprint 6502Library:1-1825027-1-TACTILE_SWITCH -> retroii_footprints:TE_1825910-6; symbol 6502:SW_PUSH_SAFE -> retroii:SW_Push
Connections:
- wire segments 121 -> 123
Changed lines of the file:
@@
 NoConn ~ 7810 5850
 $Comp
-L 6502:SW_PUSH_SAFE SW1
+L retroii:SW_Push SW1
 U 1 1 571FDFD2
 P 3580 1455
 F 0 "SW1" H 3730 1565 50  0000 C CNN
 F 1 "SW_PUSH_SAFE" H 3580 1375 50  0000 C CNN
-F 2 "6502Library:1-1825027-1-TACTILE_SWITCH" H 3580 1455 60  0001 C CNN
+F 2 "retroii_footprints:TE_1825910-6" H 3580 1455 60  0001 C CNN
 F 3 "" H 3580 1455 60  0000 C CNN
 	1    3580 1455
@@
 Wire Bus Line
 	5845 2410 6005 2410
+Wire Wire Line
+	3380 1455 3280 1455
+Wire Wire Line
+	3780 1455 3880 1455
 Wire Bus Line
 	5285 3760 5285 4890
@@
 Wire Bus Line
 	3535 3960 3535 4890
+Connection ~ 3880 1455
 $EndSCHEMATC

Commit message: finished footprints/models for power supply caps
Parts:
- C3: footprint 6502Library:C_Disc_D6_P5 -> Capacitor_THT:C_Disc_D4.7mm_W2.5mm_P5.00mm
Changed lines of the file:
@@
 F 0 "C3" H 8500 1610 50  0000 L CNN
 F 1 "1uf" H 8500 1460 50  0000 L CNN
-F 2 "6502Library:C_Disc_D6_P5" H 8490 1540 60  0001 C CNN
+F 2 "Capacitor_THT:C_Disc_D4.7mm_W2.5mm_P5.00mm" H 8490 1540 60  0001 C CNN
 F 3 "" H 8490 1540 60  0000 C CNN
 	1    8490 1540
