File: rev1.a/retroii/retroii.kicad_pcb (KiCad board)
At the start: 4 copper layers, 362 x 215.9 mm, 294 parts, among them CON1 SD_Card_SPI, J1 VGA, J10 BARREL_JACK, J11 Conn_02x10, J12 Peripheral Slot 0, J13 74LS74, J14 Game_IO_Socket, J15 Peripheral Slot 4, J16 Peripheral Slot 1, J17 Peripheral Slot 5, J18 Peripheral Slot 2, J19 Peripheral Slot 6, J2 DB9_Female_Stacked, J20 Peripheral Slot 3, J21 Peripheral Slot 7, J22 Conn_01x09, J23 Conn_01x02, J24 Headphone, J3 DB15_Female_Stacked, J6 Edge mounted connector, J7 Cassette In, J8 Cassette Out, J9 Speaker Jack, K1 PS2_KEYBOARD, K13 LM741, P1 PROP_PLUG, P2 PROP_PLUG, Q4 MPSA13, Q5 2N3904, SW1 SW_PUSH_SAFE, SW2 SPST2, SW3 SAVE, SW4 LOAD, SW5 SW_PUSH_SAFE, SW6 RESET, SW7 MISC1, SW8 MISC2, U1 74LS00, U10 74LS08, U11 LM2576-12, U12 LM2576-5, U13 LM2576-12, U14 LM2576-3.3, U15 LM2576-5, U16 Prop_P8X32A, U17 24LC256_EEPROM, U18 74LS04, U3 74LS11, U4 Prop_P8X32A, U5 24LC256_EEPROM, U6 AT28C256_EEPROM, U8 IDT7008_Dual_Port_RAM, U9 74LS32, Y1 5MHz 20pf, Y2 ECS-2100X-1MHZ, Y3 5MHz 20pf

Commit message: added m4 mounting holes
Parts:
- added H3: MountingHole, MountingHole:MountingHole_4.3mm_M4_Pad_Via, F.Cu at (549.1, 157.9)
- added H4: MountingHole, MountingHole:MountingHole_4.3mm_M4_Pad_Via, F.Cu at (233.7, 156.9)
- added H5: MountingHole, MountingHole:MountingHole_4.3mm_M4_Pad_Via, F.Cu at (550.4, 359.2)
- added H6: MountingHole, MountingHole:MountingHole_4.3mm_M4_Pad_Via, F.Cu at (231.8, 358.7)
- moved JP4 7.99 mm to (372.1, 188.5)
- moved J11 5.55 mm to (312.4, 302.1)
- moved JP2 3.74 mm to (364.9, 188.5)
- moved JP3 3.74 mm to (368.6, 186.0)
- moved J6 2.78 mm to (293.4, 312.0)
- moved J14 2.78 mm to (303.3, 312.0)
- moved P2 1.52 mm to (488.8, 171.0)
- moved R73 1.52 mm to (496.1, 168.7)
- moved R74 1.52 mm to (499.1, 168.7)
- moved R75 1.52 mm to (519.0, 168.7)
- moved R76 1.52 mm to (522.0, 168.7)
- moved R77 1.52 mm to (525.0, 168.7)
- moved R78 1.52 mm to (528.0, 168.7)
- moved R79 1.52 mm to (531.0, 168.7)
- moved R80 1.52 mm to (534.0, 168.7)
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
Commit message: finalizing edge cuts and mounting hole locations
Parts:
- moved H6 2.70 mm to (234.4, 358.2)
- moved JP14 2.32 mm to (265.4, 344.0)
- moved J3 2.32 mm to (252.6, 350.2)
- moved J2 2.32 mm to (294.3, 350.2)
- moved JP10 2.32 mm to (299.3, 344.0)
- moved JP11 2.32 mm to (302.9, 344.0)
- moved JP13 2.32 mm to (261.8, 344.0)
- moved JP9 2.32 mm to (295.7, 344.0)
- moved JP12 2.32 mm to (258.1, 344.0)
- moved C10 2.31 mm to (383.7, 351.8)
- moved J7 2.31 mm to (388.9, 356.2)
- moved J8 2.31 mm to (373.4, 356.2)
- moved H5 1.46 mm to (549.3, 358.2)
- moved H4 0.69 mm to (233.7, 157.6)
- moved H3 0.35 mm to (549.3, 157.6)
Other:
- board size 362 x 215.9 mm -> 330.2 x 215.9 mm
Changed lines of the file:
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@@
   )
   (module retroii_footprints:C_Disc_D3.0mm_W2.0mm_P2.50mm (layer F.Cu)
-    (at 386 351.75)
+    (at 383.69 351.75)
     (descr "C, Disc series, Radial, pin pitch=2.50mm, , diameter*width=3*2mm^2, Capacitor")
     (tags "C Disc series Radial pin pitch 2.50mm  diameter 3mm width 2mm Capacitor")
@@
   )
   (module retroii_footprints:SJ13525NHeadphone (layer F.Cu)
-    (at 391.25 356.25 180)
+    (at 388.94 356.25 180)
     (fp_text reference J7 (at -0.01 3.17 180) (layer F.SilkS)
       (effects (font (size 1 1) (thickness 0.15)))
@@
   )
   (module retroii_footprints:SJ13525NHeadphone (layer F.Cu)
-    (at 375.73 356.25 180)
+    (at 373.42 356.25 180)
     (fp_text reference J8 (at -5.56 3.18 180) (layer F.SilkS)
       (effects (font (size 1 1) (thickness 0.15)))
@@
   )
   (module Connector_PinHeader_2.54mm:PinHeader_1x02_P2.54mm_Vertical (layer F.Cu)
-    (at 293.355 344.01 180)
+    (at 295.675 344.01 180)
     (descr "Through hole straight pin header, 1x02, 2.54mm pitch, single row")
     (tags "Through hole pin header THT 1x02 2.54mm single row")
@@
   )
   (module Connector_PinHeader_2.54mm:PinHeader_1x02_P2.54mm_Vertical (layer F.Cu)
-    (at 296.955 344.01 180)
+    (at 299.275 344.01 180)
     (descr "Through hole straight pin header, 1x02, 2.54mm pitch, single row")
     (tags "Through hole pin header THT 1x02 2.54mm single row")
@@
   )
   (module Connector_PinHeader_2.54mm:PinHeader_1x02_P2.54mm_Vertical (layer F.Cu)
-    (at 300.555 344.01 180)
+    (at 302.875 344.01 180)
     (descr "Through hole straight pin header, 1x02, 2.54mm pitch, single row")
     (tags "Through hole pin header THT 1x02 2.54mm single row")
@@
   )
   (module Connector_PinHeader_2.54mm:PinHeader_1x02_P2.54mm_Vertical (layer F.Cu)
-    (at 255.83 344.01 180)
+    (at 258.15 344.01 180)
     (descr "Through hole straight pin header, 1x02, 2.54mm pitch, single row")
     (tags "Through hole pin header THT 1x02 2.54mm single row")
@@
   )
   (module Connector_PinHeader_2.54mm:PinHeader_1x02_P2.54mm_Vertical (layer F.Cu)
-    (at 259.43 344.01 180)
+    (at 261.75 344.01 180)
     (descr "Through hole straight pin header, 1x02, 2.54mm pitch, single row")
     (tags "Through hole pin header THT 1x02 2.54mm single row")
@@
   )
   (module Connector_PinHeader_2.54mm:PinHeader_1x02_P2.54mm_Vertical (layer F.Cu)
-    (at 263.03 344.01 180)
+    (at 265.35 344.01 180)
     (descr "Through hole straight pin header, 1x02, 2.54mm pitch, single row")
     (tags "Through hole pin header THT 1x02 2.54mm single row")
@@
   )
   (module retroii_footprints:Amphenol_L17H2220131 (layer F.Cu)
-    (at 292 350.25)
+    (at 294.32 350.25)
     (fp_text reference J2 (at -8.65 -5.11) (layer F.SilkS)
       (effects (font (size 1 1) (thickness 0.15)))
@@
   )
   (module retroii_footprints:Amphenol_L17H2440131 (layer F.Cu)
-    (at 250.29 350.25)
+    (at 252.61 350.25)
     (fp_text reference J3 (at -8.46 -5.14) (layer F.SilkS)
       (effects (font (size 1 1) (thickness 0.15)))
@@
   )
   (module MountingHole:MountingHole_4.3mm_M4_Pad_Via (layer F.Cu)
-    (at 549.08 157.86)
+    (at 549.33 157.62)
     (descr "Mounting Hole 4.3mm, M4")
     (tags "mounting hole 4.3mm m4")
@@
   )
   (module MountingHole:MountingHole_4.3mm_M4_Pad_Via (layer F.Cu)
-    (at 233.71 156.93)
+    (at 233.71 157.62)
     (descr "Mounting Hole 4.3mm, M4")
     (tags "mounting hole 4.3mm m4")
@@
   )
   (module MountingHole:MountingHole_4.3mm_M4_Pad_Via (layer F.Cu)
-    (at 550.35 359.25)
+    (at 549.33 358.2)
     (descr "Mounting Hole 4.3mm, M4")
     (tags "mounting hole 4.3mm m4")
@@
   )
   (module MountingHole:MountingHole_4.3mm_M4_Pad_Via (layer F.Cu)
-    (at 231.79 358.67)
+    (at 234.45 358.2)
     (descr "Mounting Hole 4.3mm, M4")
     (tags "mounting hole 4.3mm m4")
@@
     (pad 1 thru_hole circle (at 2.280419 -2.280419) (size 0.9 0.9) (drill 0.6) (layers *.Cu *.Mask))
   )
-  (gr_line (start 195.04 365.86) (end 556.99 365.86) (angle 90) (layer Edge.Cuts) (width 0.05))
-  (gr_line (start 195.04 149.96) (end 195.04 365.86) (angle 90) (layer Edge.Cuts) (width 0.05))
-  (gr_line (start 556.99 149.96) (end 195.04 149.96) (angle 90) (layer Edge.Cuts) (width 0.05))
+  (gr_line (start 226.79 149.96) (end 556.99 149.96) (layer Edge.Cuts) (width 0.05))
+  (gr_line (start 556.99 365.86) (end 226.79 365.86) (layer Edge.Cuts) (width 0.05))
+  (gr_line (start 226.79 365.86) (end 226.79 149.96) (layer Edge.Cuts) (width 0.05))
   (gr_line (start 556.99 365.86) (end 556.99 149.96) (angle 90) (layer Edge.Cuts) (width 0.05))
 )
